File: mac/mac.sch (KiCad schematic (older format))
At the start: 35 parts

Commit message: -выведен USB
-добавлены метки DIO
-не проверено, все ли расставлены посадочные места
Parts:
- added XP?: Вилка_PLS4, symbol elements:Вилка_PLS4
- FU?: footprint (none) -> N_RLC:Предохранитель_SMD_1812
Connections:
- net labels added: PB0, PB1, PB2, PB3, PB4, PB5, PB6, PB7, PB8, PB9, PC0_SCL1, PC1_SDA1, PC2, PE0_T2C1_DAC, PE1_T2nC1, PE2_T2C3, PE3_T2nC3, PE6_C2-RX, PE6_C2-TX, PF0_U2-RX, PF1_U2-TX, PF2_U2-En, USB_D+, USB_D-
- wire segments 126 -> 154

Commit message: на схеме (-), на трассировке (*)
-поставлен uart-rs485
-поставлена микросхема CAN
-CAN и RS выведены наружу
-выводные разъемы
*определен максимальный габарит 45х70
Parts:
- removed XP? (x2): Вилка_PLS4, symbol elements:Вилка_PLS4
- added C? (x2): 4,7мкФ(1210), N_RLC:Конденсатор_SMD_1210, symbol elements:Конденсатор_керамический
- added DD?: 5559ИН10_28(UART-RS485), symbol elements:5559ИН10_28(UART-RS485)
- added DD?: 5559ИН14А(CAN), symbol elements:5559ИН14А(CAN)
- added HL? (x20): Светодиод, N_VD_HL:Светодиод_SMD_0603, symbol elements:Светодиод
- added R? (x20): 39, N_RLC:Резистор_SMD_0805_0,125Вт, symbol elements:Резистор_0,125Вт
- added R?: 100к, N_RLC:Резистор_SMD_0805_0,125Вт, symbol elements:Резистор_0,125Вт
- added R?: 24к, N_RLC:Резистор_SMD_0805_0,125Вт, symbol elements:Резистор_0,125Вт
- added XP?: Вилка_PLS8, symbol elements:Вилка_PLS8
- added XP? (x2): Вилка_PLS10, symbol elements:Вилка_PLS10
- added XP? (x2): Вилка_PLS3, symbol elements:Вилка_PLS3
- added XP?: Вилка_PLS6, symbol elements:Вилка_PLS6
- XP?: footprint N_X:Вилка_PLS8_угловая_вертикальная -> (none)
Connections:
- net labels added: CAN_H, CAN_L, GND_LED1, GND_LED2, PD7_ADC7, RS_A, RS_B
- wire segments 154 -> 289
- no-connect marks 2 -> 5
Other:
- note added: "Выводится на \nвертикальную гребенку\nШтатно не используется"
- note added: "Выводится на\nбоковую колодку\nИспользуется штатно"
- note added: "Выводятся на боковую колодку\nИспользуются штатно"
- moved on the sheet: C1, C2, DD1, ZQ1

Commit message: трассировка в самом разгаре
выведены GPIO
не выведены ответвления на RS и CAN
не выведено программирование
не разведена земля
Parts:
- DD2, DD3: renamed from DD?; footprint (none) -> N_DD:SO-8
- XP1, XP2: renamed from XP?; footprint (none) -> N_X:Вилка_PLS8_вертикальная
- XP3, XP5, XP7: renamed from XP?; footprint (none) -> N_X:Вилка_PLS3_вертикальная
- XP4: renamed from XP?; footprint (none) -> N_X:Вилка_PLS6_вертикальная
- XP6, XP8: renamed from XP?; footprint (none) -> N_X:Вилка_PLS10_вертикальная
- gave numbers to parts that had none: 72
Connections:
- net labels added: PA4, PA5, PA6, PA7, PB10
- net labels removed: PB0, PB1, PB2, PB3, PB4
Other:
- moved on the sheet: C1, C10, C2, C3, C4, C5, C6, C7, C8, C9, DD1, FU1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

Commit message: закончена разводка, не проводилась стилистическая проверка
Parts:
- removed R13, R4, R5: 20к, N_RLC:Резистор_SMD_0805_0,125Вт, symbol elements:Резистор_0,125Вт
Connections:
- net labels added: TCK_CLK_TX, TDO_SWO, TMS_DIO_RX
- net labels removed: TCK_TX, TDI, TDO, TMS_RX, TRST
- wire segments 289 -> 278
- no-connect marks 5 -> 6
Changed lines of the file:
@@
-$EndComp
-$Comp
-L elements:Резистор_0,125Вт R5
-U 1 1 5C334333
-P 6700 10100
-F 0 "R5" V 6647 10203 60  0000 L CNN
-F 1 "20к" V 6753 10203 60  0000 L CNN
-F 2 "N_RLC:Резистор_SMD_0805_0,125Вт" H 6700 10100 60  0001 C CNN
-F 3 "" H 6700 10100 60  0001 C CNN
-	1    6700 10100
-	0    1    1    0
-$EndComp
-$Comp
-L elements:Резистор_0,125Вт R4
-U 1 1 5C33440E
-P 6350 10100
-F 0 "R4" V 6297 10203 60  0000 L CNN
-F 1 "20к" V 6403 10203 60  0000 L CNN
-F 2 "N_RLC:Резистор_SMD_0805_0,125Вт" H 6350 10100 60  0001 C CNN
-F 3 "" H 6350 10100 60  0001 C CNN
-	1    6350 10100
-	0    1    1    0
 $EndComp
 $Comp
@@
 VCC_MC
 Wire Wire Line
-	6350 9700 6350 9500
-Text Label 6350 9500 0    50   ~ 0
-VCC_MC
-Wire Wire Line
-	6700 9700 6700 9500
-Text Label 6700 9500 0    50   ~ 0
-VCC_MC
-Wire Wire Line
 	7050 9700 7050 9500
 Text Label 7050 9500 0    50   ~ 0
 VCC_MC
 Text Label 5150 10600 0    50   ~ 0
-TMS_RX
+TMS_DIO_RX
 Text Label 5150 10750 0    50   ~ 0
-TCK_TX
-Text Label 5150 10900 0    50   ~ 0
-TRST
-Text Label 5150 11050 0    50   ~ 0
-TDI
+TCK_CLK_TX
 Text Label 5150 11200 0    50   ~ 0
-TDO
+TDO_SWO
 Wire Wire Line
 	5650 10500 5650 10600
@@
 	6000 10750 5150 10750
 Wire Wire Line
-	6350 10500 6350 10900
-Connection ~ 6350 10900
-Wire Wire Line
-	6350 10900 5150 10900
-Wire Wire Line
-	6700 10500 6700 11050
-Connection ~ 6700 11050
-Wire Wire Line
-	6700 11050 5150 11050
-Wire Wire Line
 	7050 10500 7050 11200
 Connection ~ 7050 11200
 Wire Wire Line
 	7050 11200 5150 11200
-$Comp
-L elements:Вилка_PLS8 XP2
-U 1 1 5C35CF6B
-P 1850 7325
-F 0 "XP2" H 2106 7406 60  0000 C CNN
-F 1 "Вилка_PLS8" H 2100 6375 60  0001 C CNN
-F 2 "N_X:Вилка_PLS8_вертикальная" H 1850 7325 60  0001 C CNN
-F 3 "" H 1850 7325 60  0001 C CNN
-	1    1850 7325
-	1    0    0    -1
-$EndComp
 Text Label 2500 7525 0    50   ~ 0
 +3,3_prog
@@
 	2350 7925 2500 7925
 Wire Wire Line
-	2350 8025 2500 8025
-Wire Wire Line
-	2350 8125 2500 8125
-Text Label 2500 7925 0    50   ~ 0
-TRST
-Text Label 2500 8025 0    50   ~ 0
-TDI
-Text Label 2500 8125 0    50   ~ 0
-TDO
-Wire Wire Line
 	2950 2350 3275 2350
 Text Label 2500 7425 0    50   ~ 0
 +4...30
-Text Label 2500 7825 0    50   ~ 0
-TMS_RX
-Text Label 2500 7725 0    50   ~ 0
-TCK_TX
 Wire Wire Line
 	2350 6375 2500 6375
@@
 	0    1    1    0
 $EndComp
-$Comp
-L elements:Резистор_0,125Вт R13
-U 1 1 5C3BF39A
-P 13700 12100
-F 0 "R13" V 13647 12203 60  0000 L CNN
-F 1 "20к" V 13753 12203 60  0000 L CNN
-F 2 "N_RLC:Резистор_SMD_0805_0,125Вт" H 13700 12100 60  0001 C CNN
-F 3 "" H 13700 12100 60  0001 C CNN
-	1    13700 12100
-	0    1    1    0
-$EndComp
 Text Label 13550 8100 0    50   ~ 0
 GND_MC
@@
 GND_MC
 Wire Wire Line
-	13800 12650 13700 12650
-Wire Wire Line
 	13000 12650 13000 12500
 Wire Wire Line
@@
 	13350 12650 13000 12650
 Wire Wire Line
-	13700 12500 13700 12650
-Connection ~ 13700 12650
-Wire Wire Line
-	13700 12650 13350 12650
-Wire Wire Line
 	12050 11600 13000 11600
 Wire Wire Line
@@
 Wire Wire Line
 	13350 11450 13350 11700
-Wire Wire Line
-	12050 11300 13700 11300
-Wire Wire Line
-	13700 11300 13700 11700
 Text Label 12650 11600 0    50   ~ 0
 MODE
@@
 Wire Wire Line
 	6000 10750 8150 10750
-Wire Wire Line
-	6350 10900 8150 10900
-Wire Wire Line
-	6700 11050 8150 11050
 Wire Wire Line
 	7050 11200 8150 11200
@@
 Text Label 17075 8275 0    50   ~ 0
 PA4
+Text Label 2500 7825 0    50   ~ 0
+TMS_DIO_RX
+Text Label 2500 7725 0    50   ~ 0
+TCK_CLK_TX
+Text Label 2500 7925 0    50   ~ 0
+TDO_SWO
+$Comp
+L elements:Вилка_PLS8 XP2
+U 1 1 5C43CAFC
+P 1850 7325
+F 0 "XP2" H 2106 7406 60  0000 C CNN
+F 1 "Вилка_PLS8" H 2100 6375 60  0001 C CNN
+F 2 "N_X:Вилка_PLS8_вертикальная" H 1850 7325 60  0001 C CNN
+F 3 "" H 1850 7325 60  0001 C CNN
+	1    1850 7325
+	1    0    0    -1
+$EndComp
+Text Label 2500 8025 0    50   ~ 0
+RES
+Wire Wire Line
+	2500 8025 2350 8025
+NoConn ~ 2350 8125
+Wire Wire Line
+	13350 12650 13800 12650
+Wire Wire Line
+	12050 11300 13000 11300
+Wire Wire Line
+	13000 11300 13000 11600
+Connection ~ 13000 11600
 $EndSCHEMATC

Commit message: причесывание
-изменен габарит: 72х47 мм
-добавлены заливки земли на обратной стороне
-переходные отверстия вынесены за пределы контактных площадок
-прототип рекламки шелкографией
Connections:
- wire segments 278 -> 279
- no-connect marks 6 -> 5
Changed lines of the file:
@@
 L elements:Резистор_0,125Вт R6
 U 1 1 5C333E5F
-P 7050 10100
-F 0 "R6" V 6997 10203 60  0000 L CNN
-F 1 "20к" V 7103 10203 60  0000 L CNN
-F 2 "N_RLC:Резистор_SMD_0805_0,125Вт" H 7050 10100 60  0001 C CNN
-F 3 "" H 7050 10100 60  0001 C CNN
-	1    7050 10100
+P 6875 10100
+F 0 "R6" V 6822 10203 60  0000 L CNN
+F 1 "20к" V 6928 10203 60  0000 L CNN
+F 2 "N_RLC:Резистор_SMD_0805_0,125Вт" H 6875 10100 60  0001 C CNN
+F 3 "" H 6875 10100 60  0001 C CNN
+	1    6875 10100
 	0    1    1    0
 $EndComp
@@
 L elements:Резистор_0,125Вт R3
 U 1 1 5C334414
-P 6000 10100
-F 0 "R3" V 5947 10203 60  0000 L CNN
-F 1 "20к" V 6053 10203 60  0000 L CNN
-F 2 "N_RLC:Резистор_SMD_0805_0,125Вт" H 6000 10100 60  0001 C CNN
-F 3 "" H 6000 10100 60  0001 C CNN
-	1    6000 10100
+P 6500 10100
+F 0 "R3" V 6447 10203 60  0000 L CNN
+F 1 "20к" V 6553 10203 60  0000 L CNN
+F 2 "N_RLC:Резистор_SMD_0805_0,125Вт" H 6500 10100 60  0001 C CNN
+F 3 "" H 6500 10100 60  0001 C CNN
+	1    6500 10100
 	0    1    1    0
 $EndComp
@@
 L elements:Резистор_0,125Вт R2
 U 1 1 5C337872
-P 5650 10100
-F 0 "R2" V 5597 10203 60  0000 L CNN
-F 1 "20к" V 5703 10203 60  0000 L CNN
-F 2 "N_RLC:Резистор_SMD_0805_0,125Вт" H 5650 10100 60  0001 C CNN
-F 3 "" H 5650 10100 60  0001 C CNN
-	1    5650 10100
+P 6150 10100
+F 0 "R2" V 6097 10203 60  0000 L CNN
+F 1 "20к" V 6203 10203 60  0000 L CNN
+F 2 "N_RLC:Резистор_SMD_0805_0,125Вт" H 6150 10100 60  0001 C CNN
+F 3 "" H 6150 10100 60  0001 C CNN
+	1    6150 10100
 	0    1    1    0
 $EndComp
 Wire Wire Line
-	5650 9700 5650 9500
-Text Label 5650 9500 0    50   ~ 0
+	6150 9700 6150 9500
+Text Label 6150 9500 0    50   ~ 0
 VCC_MC
 Wire Wire Line
-	6000 9700 6000 9500
-Text Label 6000 9500 0    50   ~ 0
+	6500 9700 6500 9500
+Text Label 6500 9500 0    50   ~ 0
 VCC_MC
 Wire Wire Line
-	7050 9700 7050 9500
-Text Label 7050 9500 0    50   ~ 0
+	6875 9700 6875 9500
+Text Label 6875 9500 0    50   ~ 0
 VCC_MC
 Text Label 5150 10600 0    50   ~ 0
@@
 TDO_SWO
 Wire Wire Line
-	5650 10500 5650 10600
-Connection ~ 5650 10600
-Wire Wire Line
-	5650 10600 5150 10600
-Wire Wire Line
-	6000 10500 6000 10750
-Connection ~ 6000 10750
-Wire Wire Line
-	6000 10750 5150 10750
-Wire Wire Line
-	7050 10500 7050 11200
-Connection ~ 7050 11200
-Wire Wire Line
-	7050 11200 5150 11200
+	6150 10500 6150 10600
+Wire Wire Line
+	6500 10500 6500 10750
+Wire Wire Line
+	6875 10500 6875 11200
 Text Label 2500 7525 0    50   ~ 0
 +3,3_prog
@@
 Wire Wire Line
 	2350 9175 2500 9175
+Text Label 2500 9175 0    50   ~ 0
+VCC_MC
 Text Label 2500 8975 0    50   ~ 0
-VCC_MC
-Text Label 2500 9175 0    50   ~ 0
 GND_MC
 Text Label 7350 11350 0    50   ~ 0
@@
 Wire Wire Line
 	8150 12700 7350 12700
-Wire Wire Line
-	5650 10600 8150 10600
-Wire Wire Line
-	6000 10750 8150 10750
-Wire Wire Line
-	7050 11200 8150 11200
 Text Label 7350 10000 0    50   ~ 0
 PC0_SCL1
@@
 Wire Wire Line
 	2500 8025 2350 8025
-NoConn ~ 2350 8125
 Wire Wire Line
 	13350 12650 13800 12650
@@
 	13000 11300 13000 11600
 Connection ~ 13000 11600
+Connection ~ 6150 10600
+Wire Wire Line
+	6150 10600 8150 10600
+Connection ~ 6500 10750
+Wire Wire Line
+	6500 10750 8150 10750
+Connection ~ 6875 11200
+Wire Wire Line
+	6875 11200 8150 11200
+Wire Wire Line
+	5150 10600 6150 10600
+Wire Wire Line
+	5150 10750 6500 10750
+Wire Wire Line
+	5150 11200 6875 11200
+Text Label 2500 8125 0    50   ~ 0
+GND
+Wire Wire Line
+	2350 8125 2500 8125
 $EndSCHEMATC

Commit message: "mac" версия 1
Parts:
- removed C1, C2: 12пФ(0603), N_RLC:Конденсатор_SMD_0603, symbol elements:Конденсатор_керамический
- removed C10, C3, C4, C5, C6, C7, C8, C9: 4,7мкФ(1210), N_RLC:Конденсатор_SMD_1210, symbol elements:Конденсатор_керамический
- removed DD1: 1986ВЕ92QL, N_DD:Микросхема_1986ВЕ92QL, symbol elements:1986ВЕ92QL
- removed DD2: 5559ИН14А(CAN), N_DD:SO-8, symbol elements:5559ИН14А(CAN)
- removed DD3: 5559ИН10_28(UART-RS485), N_DD:SO-8, symbol elements:5559ИН10_28(UART-RS485)
- removed FU1: Предохранитель, N_RLC:Предохранитель_SMD_1812, symbol elements:Предохранитель
- removed G1: стабилизатор_нерегулируемый_LM2950, N_G:Стабилизатор_корпус_TO-92, symbol elements:стабилизатор_нерегулируемый_LM2950
- removed HL1, HL10, HL11, HL12, HL13, HL14, HL15, HL16, HL17, HL18, HL19, HL2, HL20, HL21, HL3, HL4, HL5, HL6, HL7, HL8, HL9: Светодиод, N_VD_HL:Светодиод_SMD_0603, symbol elements:Светодиод
- removed L1, L2, L3, L4: 33мкГн(0805), N_RLC:Чип-индуктивность_SMD_0805, symbol elements:Чип-индуктивность
- removed R1, R14, R15, R16, R17, R18, R19, R20, R21, R22, R23, R24, R25, R26, R27, R28, R29, R30, R31, R32, R33: 39, N_RLC:Резистор_SMD_0805_0,125Вт, symbol elements:Резистор_0,125Вт
- removed R10, R11, R12, R2, R3, R6, R7: 20к, N_RLC:Резистор_SMD_0805_0,125Вт, symbol elements:Резистор_0,125Вт
- removed R8: 100к, N_RLC:Резистор_SMD_0805_0,125Вт, symbol elements:Резистор_0,125Вт
- removed R9: 24к, N_RLC:Резистор_SMD_0805_0,125Вт, symbol elements:Резистор_0,125Вт
- removed VD1, VD2, VD3, VD4: BAR43CFILM, N_VD_HL:Диод_BAR43CFILM_SOT-23, symbol elements:Диод_шоттки
- removed XP1, XP2: Вилка_PLS8, N_X:Вилка_PLS8_вертикальная, symbol elements:Вилка_PLS8
- removed XP3, XP5, XP7: Вилка_PLS3, N_X:Вилка_PLS3_вертикальная, symbol elements:Вилка_PLS3
- removed XP4: Вилка_PLS6, N_X:Вилка_PLS6_вертикальная, symbol elements:Вилка_PLS6
- removed XP6, XP8: Вилка_PLS10, N_X:Вилка_PLS10_вертикальная, symbol elements:Вилка_PLS10
- removed ZQ1: 16М, N_RLC:Резонатор_РК456МДУ(DIP), symbol elements:Резонатор_кварцевый
- added DD?: 1986ВЕ92QL, N_DD:Микросхема_1986ВЕ92QL, symbol elements:1986ВЕ92QL
Connections:
- net labels removed: +3,3, +3,3_prog, +4...30, A_GND_MC, A_VCC_MC, CAN_H, CAN_L, GND, GND_LED1, GND_LED2, GND_MC, MODE, PA4, PA5, PA6, PA7, PB10, PB5, PB6, PB7, PB8, PB9, PC0_SCL1, PC1_SDA1, PC2, PD5_ADC5, PD6_ADC6, PD7_ADC7, PE0_T2C1_DAC, PE1_T2nC1, PE2_T2C3, PE3_T2nC3, PE6_C2-RX, PE6_C2-TX, PF0_U2-RX, PF1_U2-TX, PF2_U2-En, RES, RS_A, RS_B, TCK_CLK_TX, TDO_SWO, TMS_DIO_RX, USB_D+, USB_D-, VCC, VCC_MC
- wire segments 279 -> 0
- no-connect marks 5 -> 0
Other:
- note removed: "Выводится на \nвертикальную гребенку\nШтатно не используется"
- note removed: "Выводится на\nбоковую колодку\nИспользуется штатно"
- note removed: "Выводятся на боковую колодку\nИспользуются штатно"

Commit message: не размещены вилки, определен габарит
Parts:
- added C1, C2, C3, C4, C5, C6, C7, C8, C9: Конденсатор_керамический, N_RLC:Конденсатор_SMD_0603, symbol elements:Конденсатор_керамический
- added R1, R2, R3, R4, R5, R6, R7, R8: Резистор_0,065Вт, N_RLC:Резистор_SMD_0603_0,065_Вт, symbol elements:Резистор_0,065Вт
- added VD1: Диод_S13, N_VD_HL:Диод_S13_SOD-123, symbol elements:Диод_шоттки
- added VD2, VD3: Диоды_шоттки_BAT54S, N_VD_HL:Транзистор_IRLML6344TR_SOT-23, symbol elements:Диоды_шоттки_BAT54S
- added XP1: Вилка_PLD6_ПРОГ_STM, N_X:Вилка_PLD6_вертикальная, symbol elements:Вилка_PLD6_ПРОГ_STM
- added ZQ1: Резонатор_16МГц, N_RLC:Резонатор_РК456МДУ(DIP), symbol elements:Резонатор_кварцевый
- gave numbers to parts that had none: 1
Connections:
- net 3V: now reaches DD1.1 (DUcc)
- net 3V: now also DD1.12 (DUcc), DD1.24 (AUcc1), DD1.28 (AUcc), DD1.38 (DUcc), DD1.48 (DUcc), C2.1, C3.1, C6.1, C7.1, C8.1, C9.1, R1.1, R2.1, R3.2, R8.1, VD1.2, VD2.2, VD3.2
- net USB_D-: now reaches DD1.10 (DN)
- net USB_D-: now also R7.2
- net gnd: now reaches DD1.11 (DGND)
- net gnd: now also DD1.23 (AGND1), DD1.27 (AGND), DD1.39 (DGND), DD1.49 (DGND), DD1.64 (DGND), C1.2, C2.2, C3.2, C4.2, C5.1, C6.2, C7.2, C8.2, C9.2, R4.2, R5.2, VD2.1, VD3.1, XP1.6 (GND)
- net BUcc: now reaches DD1.13 (BUcc)
- net BUcc: now also C1.1, R8.2
- net PE6_T3C3: now reaches DD1.16 (PE6)
- net RESET: now reaches DD1.18 (RESET)
- net RESET: now also R3.1, XP1.5 (RST)
- net at DD1.19 (OSC_IN): now also C4.1, ZQ1.1
- net at DD1.20 (OSC_OUT): now also C5.2, ZQ1.2
- net PE1_DAC2_REF: now reaches DD1.25 (PE1/DAC2_REF)
- net PE0_DAC2_OUT: now reaches DD1.26 (PE0/DAC2_OUT)
- net PD7_ADC7: now reaches DD1.29 (PD7)
- net PD4_ADC4: now reaches DD1.30 (PD4(JB_TDO))
- net UART2_RX_TMS: now reaches DD1.31 (PD0(JB_TMS)/RX101)
- net UART2_RX_TMS: now also R2.2, XP1.4 (DIO)
- net UART2_TX_TCK: now reaches DD1.32 (PD1(JB_TCK)/TX101)
- net UART2_TX_TCK: now also R1.2, XP1.3 (SLK)
- net PD2_ADC2: now reaches DD1.33 (PD2(JB_TRST))
- net PD3_ADC3: now reaches DD1.34 (PD3(JB_TDI))
- net PD5_ADC5: now reaches DD1.35 (PD5)
- net PD6_ADC6: now reaches DD1.36 (PD6)
- net PF2_CAN2_RX: now reaches DD1.4 (PF2)
- net PC2_UART2_EN: now reaches DD1.40 (PC2)
- net PC1_SDA1: now reaches DD1.41 (PC1)
- net PC0_SCL1: now reaches DD1.42 (PC0)
- net PB0_T3C1: now reaches DD1.43 (PB0(JA_TDO))
- net PB1_T3C1n: now reaches DD1.44 (PB1(JA_TMS))
- net PB2_CAN1_TX: now reaches DD1.45 (PB2(JA_TCK))
- net PB3CAN1_RX: now reaches DD1.46 (PB3(JA_TDI))
- net PB4_UART1_en: now reaches DD1.47 (PB4(JA_TRST))
- net PF3_CAN2_TX: now reaches DD1.5 (PF3)
- net PB5_UART1_TX: now reaches DD1.50 (PB5)
- net PB6_UART1_RX: now reaches DD1.51 (PB6)
- net PB7_T3C4: now reaches DD1.52 (PB7)
- net PB8_T3C4n: now reaches DD1.53 (PB8)
- net PA7: now reaches DD1.56 (PA7)
- net PA6: now reaches DD1.57 (PA6)
- net PA5_T1C3: now reaches DD1.58 (PA5)
- net PA4_T1C2n: now reaches DD1.59 (PA4)
- net mode_101: now reaches DD1.6 (PF4(MODE[0]))
- net mode_101: now also DD1.8 (PF6(MODE[2])), R4.1, XP1.1 (mode)
- net PA3_T1C2: now reaches DD1.60 (PA3)
- net PA2_T1C1n: now reaches DD1.61 (PA2)
- net PA1_T1C1: now reaches DD1.62 (PA1)
- net PA0: now reaches DD1.63 (PA0)
- net mode_010: now reaches DD1.7 (PF5(MODE[1]))
- net mode_010: now also R5.1
- net USB_D+: now reaches DD1.9 (DP)
- net USB_D+: now also R6.2
- new net: R6.1, VD2.3
- new net: VD1.1, XP1.2 (3V)
- new net: R7.1, VD3.3
- no-connect marks 0 -> 5
Other:
- moved on the sheet: DD1
